File: STM32F103C8T6-breakout-board_compact.brd (EAGLE design)
At the start: 21.6 x 55.2 mm, 37 parts, among them J3 AVX_6-PIN_009159006061916, J4 CORTEX_DEBUG_PTH, J5 10118194-0001LF, U1 STM32F103C8T6, U2 CJT1117-3.3-SOT223

Commit message: Updated files.
Parts:
- added L1: 470R-2A, OPL_Ferrite_and_Magnetic_Bead:L0805
- J1, J2: device SparkFun-Connectors:1X19_NO_SILK -> SparkFun-Connectors:1X20_NOSILK
- moved C7 2.84 mm to (6.35, 36.2), turned to 180 degrees
- moved J6 1.91 mm to (10.8, 53.3)
- moved J8 1.91 mm to (5.71, 44.5)
- moved LED1 1.91 mm to (3.81, 54.0)
- moved LED2 1.91 mm to (5.71, 54.0)
- moved R3 1.91 mm to (15.9, 47.0)
- moved R4 1.91 mm to (8.26, 54.0)
- moved R5 1.91 mm to (12.1, 47.0), turned to 180 degrees
- moved R6 1.91 mm to (8.26, 50.2)
- moved R7 1.91 mm to (3.81, 50.2)
- moved R8 1.91 mm to (5.71, 50.2)
- moved J1 1.90 mm to (1.91, 55.2)
- moved J2 1.90 mm to (19.7, 55.2)
- moved J7 1.90 mm to (10.8, 50.8)
- moved C6 1.27 mm to (6.35, 37.5), turned to 180 degrees
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Connections:
- new net AVDD: C6.1, C7.1, J2.2, L1.1, U1.9
- net BOOT1*: now also J1.7
- net GND: now also J2.18; no longer J2.17
- net JTDI*: now also J2.14; no longer J2.13
- net JTRST*: now also J2.13; no longer J2.12
- net NRST: now also J2.15; no longer J2.14
- net PA0: now also J2.5; no longer J2.4
- net PA1: now also J2.4; no longer J2.3
- net PA10*: now also J1.16; no longer J1.15
- net PA2: now also J2.3; no longer J2.2
- net PA8*: now also J1.14; no longer J1.13
- net PA9*: now also J1.15; no longer J1.14
- net PB10*: now also J1.8; no longer J1.7
- net PB11*: now also J1.9; no longer J1.8
- net PB12*: now also J1.10; no longer J1.9
- net PB13*: now also J1.11; no longer J1.10
- net PB14*: now also J1.12; no longer J1.11
- net PB15*: now also J1.13; no longer J1.12
- net PB5: now also J2.12; no longer J2.11
- net PB6*: now also J2.11; no longer J2.10
- net PB7*: now also J2.10; no longer J2.9
- net PB8*: now also J2.9; no longer J2.8
- net PB9*: now also J2.8; no longer J2.7
- net PC13: now also J2.6; no longer J2.5
- net SWCLK*: now also J2.19; no longer J2.18
- net SWDIO*: now also J2.17; no longer J2.16
- net SWO*: now also J2.16; no longer J2.15
- net USB_DM*: now also J1.18; no longer J1.17
- net USB_DP*: now also J1.19; no longer J1.18
- net VBAT_1.8-3.6V: now also J2.7; no longer J2.6
- net VDD: now also J2.20, L1.2; no longer C6.1, C7.1, J2.19, U1.9
- net VIN_4.8-15V: now also J1.17; no longer J1.16
- net VUSB: now also J1.20; no longer J1.19
Routing:
- net AVDD: track 0.00 -> 27.5 mm, vias 0 -> 1
- net BOOT1*: track 17.2 -> 32.2 mm
- net PA3: track 38.0 -> 42.0 mm
- net VDD: track 30.9 -> 27.2 mm
- net PB1: track 12.1 -> 14.7 mm
- net PA7: track 16.1 -> 18.6 mm
- net PB0: track 14.1 -> 16.6 mm
- net PA6: track 18.0 -> 20.6 mm
- net PA5: track 20.0 -> 22.5 mm
- net BOOT0: track 14.7 -> 17.3 mm
- net PA4: track 22.0 -> 24.5 mm
- net SWDIO*: track 40.2 -> 39.5 mm
- net USB_DP*: track 30.2 -> 29.6 mm
- net SWCLK*: track 44.2 -> 43.6 mm
- net OSC_IN: track 2.17 -> 2.81 mm
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Other:
- board size 21.6 x 55.2 mm -> 21.6 x 57.1 mm
- board text added: "-------POWER------- VDD/AVDD: 2-3.6V. Must be 3.3V if C39- 097/C387- 415 are used for Q1/Q2. VUSB: 5V from USB1 VIN: 4.8-15V BAT: 1.8-3.6V. Short R2 if unused. **WARNING**: Do NOT power MCU from VDD if EITHER VIN or USB1 are also being used. --------GPIO-------- Max current, ea pin: 25 mA Max current, total: 150 mA OUT (minus MCU power, ~7 -50 mA) and 150 mA IN (minus MCU po- wer) Bar on pin labe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"
- board text added: "AVDD"
- board text added: "B2"
- board text removed: "-------POWER------- VDD: 2-3.6V. Must be 3.3V if C39097/ C387415 are used for Q1/Q2. VUSB: 5V from USB1 VIN: 4.8-15V BAT: 1.8-3.6V. Short R2 if unused. **WARNING**: Do NOT power MCU from VDD if EITHER VIN or USB1 are also being used. --------GPIO-------- Max current, ea pin: 25 mA Max current, total: 150 mA OUT (minus MCU power, ~7 -50 mA) and 150 mA IN (minus MCU power) Hor. bar = 5V tolerant pi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"
- board text removed: "~RST"
